Commit message: Added camera keypoint of the camera (with orientation). This is useful for perception rewards

File: source/Racing_Quadcopter/Racing_Quadcopter/assets/robots/anemos/anemos.urdf (robot description, URDF)
Before this commit: robot drone_acc_mass, 5 links, 4 joints
Links:
- added link camera_keypoint, mass 1e-9
Joints:
- added joint camera_keypoint_fixed: type fixed, parent base_link, child camera_keypoint, origin xyz=0.085196 0.001872 0.067774 rpy=0 -0.523599 0

Commit message: fix(urdf): dummy visual to resolve USD reference
Add dummy visual to camera_keypoint to resolve USD reference.
The initial error occured because a camera_keypoint was added
without it. The original URDF is not flawed, it was our URDF only.

File: source/Racing_Quadcopter/Racing_Quadcopter/assets/robots/anemos/anemos.urdf (robot description, URDF)
Before this commit: robot drone_acc_mass, 6 links, 5 joints
Links:
- link camera_keypoint: geometry visual sphere radius=0.001
